Commit message: Update Franka robot configuration: add finger joint and adjust RViz settings

File: franka_description/end_effectors/common/franka_hand.xacro (robot description, xacro)
@@ -118,5 +118,5 @@
       <axis xyz="0 -1 0" />
       <limit effort="100" lower="0.0" upper="0.04" velocity="0.2" />
-      <mimic joint="${ee_prefix}finger_joint1" />
+      <!-- <mimic joint="${ee_prefix}finger_joint1" /> -->
       <dynamics damping="0.3" />
     </joint>

File: franka_description/robots/common/franka_arm.ros2_control.xacro (robot description, xacro)
@@ -66,4 +66,5 @@
       <xacro:if value="${gazebo and hand}">
         <xacro:configure_joint joint_name="${arm_id}_finger_joint1" initial_position="0.0" />
+        <xacro:configure_joint joint_name="${arm_id}_finger_joint2" initial_position="0.0" />
       </xacro:if>
     </ros2_control>
